File: design/electrical/gps_can_v0.1.sch (KiCad schematic (older format))
At the start: 24 parts, among them IC1 ATMEGA16M1-A, J1 SMA, U1 TPS2030, U2 LM1117-3.3, U3 RXM-GPS-RM, U4 ADG787, U5 ATA6561, U6 ATA6561

Commit message: Removed voltage divider on GPS_RX, pullup resistor ~RESET for GPS and S3 & S4 as +5V supply. Added pullup resistor for ~GPS_OC. Solved most ERC errors.
Parts:
- removed R3: 10k, Resistors_SMD:R_0603_HandSoldering, symbol R_Small
- removed R4: 20k, Resistors_SMD:R_0603_HandSoldering, symbol R_Small
- removed R9: DNP, Resistors_SMD:R_0603_HandSoldering, symbol R_Small
- R7: value DNP -> 0
- R8: value 0 -> DNP
Connections:
- net labels added: ALT_5V, GNDPWR
- net labels removed: GPS_RX, S3, S4
- wire segments 146 -> 136
- no-connect marks 0 -> 118
Other:
- moved on the sheet: U1
