File: design/electrical/gps_can_v0.1.kicad_pcb (KiCad board)
At the start: 2 copper layers, 90.2 x 95.9 mm, 24 parts, among them IC1 ATMEGA16M1-A, J1 SMA, U1 TPS2030, U2 LM1117-3.3, U3 RXM-GPS-RM, U4 ADG787, U5 ATA6561, U6 ATA6561

Commit message: Updated PCB layout and Gerbers
Parts:
- removed R3: 10k, Resistors_SMD:R_0603_HandSoldering
- removed R4: 20k, Resistors_SMD:R_0603_HandSoldering
- removed R9: DNP, Resistors_SMD:R_0603_HandSoldering
- R7: value DNP -> 0
- R8: value 0 -> DNP
- moved R1 19.9 mm to (106.7, 88.9), turned to 0 degrees
- moved R8 14.6 mm to (111.1, 71.1)
- moved R7 14.0 mm to (109.2, 71.1)
Connections:
- net /5V_BUS renamed 5V_BUS
- net /CAN1_STBY renamed CAN1_STBY
- net /CAN2_STBY renamed CAN2_STBY
- net /CAN_SEL renamed CAN_SEL
- net /GPS_EN renamed GPS_EN
- net /GPS_RX renamed Net-(IC1-Pad2)
- net /GPS_TX renamed GPS_TX
- net /RX_CAN renamed RX_CAN
- net /TX_CAN renamed TX_CAN
- H2 pad 39: /S3 -> Net-(H2-Pad39)
- H2 pad 40: /S3 -> Net-(H2-Pad40)
- H2 pad 41: /S4 -> Net-(H2-Pad41)
- H2 pad 42: /S4 -> Net-(H2-Pad42)
- IC1 pad 25: /~GPS_OC -> ~GPS_OC
- R1 pad 1: Net-(C1-Pad1) -> +5V
- R1 pad 2: Net-(R1-Pad2) -> ~GPS_OC
- R8 pad 2: /S3 -> ALT_5V
- U1 pad 5: /~GPS_OC -> ~GPS_OC
- U3 pad 8: Net-(R1-Pad2) -> Net-(U3-Pad8)
Routing:
- net Net-(IC1-Pad2): track 49.8 -> 6.88 mm
- net /S4: track 31.4 -> 0.00 mm
- net /S3: track 28.0 -> 0.00 mm, vias 1 -> 0
- net ~GPS_OC: track 0.00 -> 26.6 mm
- net /~GPS_OC: track 24.6 -> 0.00 mm
- net 5V_BUS: track 47.0 -> 32.9 mm
- net +5V: track 171.2 -> 161.5 mm
- net Net-(R1-Pad2): track 7.81 -> 0.00 mm
- net Net-(U3-Pad5): track 6.06 -> 0.00 mm
- net GND: track 152.2 -> 148.9 mm
- net Net-(C1-Pad1): track 32.9 -> 29.7 mm
