File: design/electrical/gps_module.sch (KiCad schematic (older format))
At the start: 21 parts, among them IC1 ATMEGA16M1-A, J1 SMA, U1 TPS2030, U2 LM1117-3.3, U3 RXM-GPS-RM, U4 ADG787, U5 ATA6561, U6 ATA6561

Commit message: add 3v3 converter and LEDs
Parts:
- removed R8: DNP, Resistors_SMD:R_0603_HandSoldering, symbol R_Small
- added C3, C4, C5: 1uF, Capacitors_SMD:C_0603, symbol C_Small
- added D2, D3, D4: Led_Small, LEDs:LED_0805, symbol Led_Small
- added P2: CONN_01X04, Connectors_JST:JST_GH_BM04B-GHS-TBT_04x1.25mm_Straight, symbol CONN_01X04
- added R3, R4: 1k, Resistors_SMD:R_0603_HandSoldering, symbol R_Small
- added U7: LM1117-3.3, TO_SOT_Packages_SMD:SOT-223, symbol LM1117-3.3
- C1, C2: footprint Capacitors_SMD:C_1210_HandSoldering -> Capacitors_SMD:C_0603
- L1: footprint Inductors:Inductor_Taiyo-Yuden_NR-24xx_HandSoldering -> Capacitors_SMD:C_0603
- R7: value 0 -> 1k
Connections:
- net labels added: +3.3V, 3V3_GPS
- net labels removed: ALT_5V, GNDPWR
- wire segments 136 -> 155
- no-connect marks 118 -> 116
Other:
- moved on the sheet: C1
